File: src/elec/myrt-charging_stations.sch (KiCad schematic (older format))
At the start: 15 parts

Commit message: Start PCB design
Parts:
- D3, D4, D5: renamed from D?; footprint (none) -> LEDs:LED-5MM; symbol LED -> LED-RESCUE-myrt
- P10, P11, P6, P7, P8, P9: renamed from P?; footprint (none) -> Connect:bornier2
- R3, R4, R5, R6: renamed from R?; footprint (none) -> Resistors_ThroughHole:Resistor_Horizontal_RM10mm
- R7, R8: renamed from R?; footprint (none) -> Resistors_ThroughHole:Resistor_Horizontal_RM30mm
Connections:
- wire segments 30 -> 24
Changed lines of the file:
@@
 EESchema Schematic File Version 2
+LIBS:myrt-rescue
 LIBS:power
 LIBS:device
@@
 LIBS:contrib
 LIBS:valves
-LIBS:borniers
-LIBS:con_p
-LIBS:dips-s
-LIBS:K-module
-LIBS:KubiackLIB
-LIBS:MSP430
-LIBS:opto_p
-LIBS:pololu_a4988
-LIBS:RovingNetworks
-LIBS:sparkfun
-LIBS:stepper drivers
-LIBS:texas_p
-LIBS:arduino
 LIBS:myrt-cache
 EELAYER 25 0
@@
 $EndDescr
 $Comp
-L CONN_2 P?
+L CONN_2 P7
 U 1 1 591C7A4B
 P 4800 3600
-F 0 "P?" V 4750 3600 40  0000 C CNN
+F 0 "P7" V 4750 3600 40  0000 C CNN
 F 1 "CONN_2" V 4850 3600 40  0000 C CNN
-F 2 "" H 4800 3600 60  0001 C CNN
+F 2 "Connect:bornier2" H 4800 3600 60  0001 C CNN
 F 3 "" H 4800 3600 60  0001 C CNN
 	1    4800 3600
@@
 $EndComp
 $Comp
-L LED D?
+L LED-RESCUE-myrt D4
 U 1 1 591C7B22
 P 5850 3250
-F 0 "D?" H 5850 3350 50  0000 C CNN
+F 0 "D4" H 5850 3350 50  0000 C CNN
 F 1 "Yellow" H 5850 3150 50  0000 C CNN
-F 2 "" H 5850 3250 50  0001 C CNN
+F 2 "LEDs:LED-5MM" H 5850 3250 50  0001 C CNN
 F 3 "" H 5850 3250 50  0001 C CNN
 	1    5850 3250
@@
 $EndComp
 $Comp
-L CONN_2 P?
+L CONN_2 P10
 U 1 1 591C7D17
 P 7000 3600
-F 0 "P?" V 6950 3600 40  0000 C CNN
+F 0 "P10" V 6950 3600 40  0000 C CNN
 F 1 "CONN_2" V 7050 3600 40  0000 C CNN
-F 2 "" H 7000 3600 60  0001 C CNN
+F 2 "Connect:bornier2" H 7000 3600 60  0001 C CNN
 F 3 "" H 7000 3600 60  0001 C CNN
 	1    7000 3600
@@
 Power input\nFrom energy storage station
 Wire Wire Line
-	5150 3700 6100 3700
-Wire Wire Line
-	6100 3700 6650 3700
-Wire Wire Line
-	5150 3500 5300 3500
-Wire Wire Line
-	5300 3500 6200 3500
+	5150 3700 6650 3700
+Wire Wire Line
+	5150 3500 6200 3500
 Text Label 5500 3700 0    60   ~ 0
 POWER_GND
@@
 POWER_5V
 $Comp
-L R R?
+L R R7
 U 1 1 591C8302
 P 6350 3500
-F 0 "R?" V 6430 3500 50  0000 C CNN
+F 0 "R7" V 6430 3500 50  0000 C CNN
 F 1 "100Ω 0.5W" V 6250 3500 50  0000 C CNN
-F 2 "" V 6280 3500 50  0001 C CNN
+F 2 "Resistors_ThroughHole:Resistor_Horizontal_RM30mm" V 6280 3500 50  0001 C CNN
 F 3 "" H 6350 3500 50  0001 C CNN
 	1    6350 3500
@@
 	6650 3500 6500 3500
 $Comp
-L R R?
+L R R4
 U 1 1 591C834C
 P 5500 3250
-F 0 "R?" V 5580 3250 50  0000 C CNN
+F 0 "R4" V 5580 3250 50  0000 C CNN
 F 1 "470" V 5500 3250 50  0000 C CNN
-F 2 "" V 5430 3250 50  0001 C CNN
+F 2 "Resistors_ThroughHole:Resistor_Horizontal_RM10mm" V 5430 3250 50  0001 C CNN
 F 3 "" H 5500 3250 50  0001 C CNN
 	1    5500 3250
@@
 Status display led
 $Comp
-L CONN_2 P?
+L CONN_2 P6
 U 1 1 591C929A
 P 4800 2450
-F 0 "P?" V 4750 2450 40  0000 C CNN
+F 0 "P6" V 4750 2450 40  0000 C CNN
 F 1 "CONN_2" V 4850 2450 40  0000 C CNN
-F 2 "" H 4800 2450 60  0001 C CNN
+F 2 "Connect:bornier2" H 4800 2450 60  0001 C CNN
 F 3 "" H 4800 2450 60  0001 C CNN
 	1    4800 2450
@@
 $EndComp
 $Comp
-L LED D?
+L LED-RESCUE-myrt D3
 U 1 1 591C92A0
 P 5850 2100
-F 0 "D?" H 5850 2200 50  0000 C CNN
+F 0 "D3" H 5850 2200 50  0000 C CNN
 F 1 "Green" H 5850 2000 50  0000 C CNN
-F 2 "" H 5850 2100 50  0001 C CNN
+F 2 "LEDs:LED-5MM" H 5850 2100 50  0001 C CNN
 F 3 "" H 5850 2100 50  0001 C CNN
 	1    5850 2100
@@
 $EndComp
 $Comp
-L CONN_2 P?
+L CONN_2 P9
 U 1 1 591C92A6
 P 7000 2450
-F 0 "P?" V 6950 2450 40  0000 C CNN
+F 0 "P9" V 6950 2450 40  0000 C CNN
 F 1 "CONN_2" V 7050 2450 40  0000 C CNN
-F 2 "" H 7000 2450 60  0001 C CNN
+F 2 "Connect:bornier2" H 7000 2450 60  0001 C CNN
 F 3 "" H 7000 2450 60  0001 C CNN
 	1    7000 2450
@@
 Power output\nTo copper contacts
 Wire Wire Line
-	5150 2550 6100 2550
-Wire Wire Line
-	6100 2550 6650 2550
-Wire Wire Line
-	5150 2350 5300 2350
-Wire Wire Line
-	5300 2350 6200 2350
+	5150 2550 6650 2550
+Wire Wire Line
+	5150 2350 6200 2350
 Text Label 5500 2550 0    60   ~ 0
 POWER_GND
@@
 POWER_5V
 $Comp
-L R R?
+L R R6
 U 1 1 591C92B3
 P 6350 2350
-F 0 "R?" V 6430 2350 50  0000 C CNN
+F 0 "R6" V 6430 2350 50  0000 C CNN
 F 1 "500Ω 0.1W" V 6250 2350 50  0000 C CNN
-F 2 "" V 6280 2350 50  0001 C CNN
+F 2 "Resistors_ThroughHole:Resistor_Horizontal_RM10mm" V 6280 2350 50  0001 C CNN
 F 3 "" H 6350 2350 50  0001 C CNN
 	1    6350 2350
@@
 	6650 2350 6500 2350
 $Comp
-L R R?
+L R R3
 U 1 1 591C92BA
 P 5500 2100
-F 0 "R?" V 5580 2100 50  0000 C CNN
+F 0 "R3" V 5580 2100 50  0000 C CNN
 F 1 "470" V 5500 2100 50  0000 C CNN
-F 2 "" V 5430 2100 50  0001 C CNN
+F 2 "Resistors_ThroughHole:Resistor_Horizontal_RM10mm" V 5430 2100 50  0001 C CNN
 F 3 "" H 5500 2100 50  0001 C CNN
 	1    5500 2100
@@
 Medium charging station (50mA)
 $Comp
-L CONN_2 P?
+L CONN_2 P8
 U 1 1 591C9885
 P 4800 4700
-F 0 "P?" V 4750 4700 40  0000 C CNN
+F 0 "P8" V 4750 4700 40  0000 C CNN
 F 1 "CONN_2" V 4850 4700 40  0000 C CNN
-F 2 "" H 4800 4700 60  0001 C CNN
+F 2 "Connect:bornier2" H 4800 4700 60  0001 C CNN
 F 3 "" H 4800 4700 60  0001 C CNN
 	1    4800 4700
@@
 $EndComp
 $Comp
-L LED D?
+L LED-RESCUE-myrt D5
 U 1 1 591C988B
 P 5850 4350
-F 0 "D?" H 5850 4450 50  0000 C CNN
+F 0 "D5" H 5850 4450 50  0000 C CNN
 F 1 "Red" H 5850 4250 50  0000 C CNN
-F 2 "" H 5850 4350 50  0001 C CNN
+F 2 "LEDs:LED-5MM" H 5850 4350 50  0001 C CNN
 F 3 "" H 5850 4350 50  0001 C CNN
 	1    5850 4350
@@
 $EndComp
 $Comp
-L CONN_2 P?
+L CONN_2 P11
 U 1 1 591C9891
 P 7000 4700
-F 0 "P?" V 6950 4700 40  0000 C CNN
+F 0 "P11" V 6950 4700 40  0000 C CNN
 F 1 "CONN_2" V 7050 4700 40  0000 C CNN
-F 2 "" H 7000 4700 60  0001 C CNN
+F 2 "Connect:bornier2" H 7000 4700 60  0001 C CNN
 F 3 "" H 7000 4700 60  0001 C CNN
 	1    7000 4700
@@
 $EndComp
 Wire Wire Line
-	5150 4800 6100 4800
-Wire Wire Line
-	6100 4800 6650 4800
-Wire Wire Line
-	5150 4600 5300 4600
-Wire Wire Line
-	5300 4600 6200 4600
+	5150 4800 6650 4800
+Wire Wire Line
+	5150 4600 6200 4600
 Text Label 5500 4800 0    60   ~ 0
 POWER_GND
@@
 POWER_5V
 $Comp
-L R R?
+L R R8
 U 1 1 591C989D
 P 6350 4600
-F 0 "R?" V 6430 4600 50  0000 C CNN
+F 0 "R8" V 6430 4600 50  0000 C CNN
 F 1 "33Ω 1.5W" V 6250 4600 50  0000 C CNN
-F 2 "" V 6280 4600 50  0001 C CNN
+F 2 "Resistors_ThroughHole:Resistor_Horizontal_RM30mm" V 6280 4600 50  0001 C CNN
 F 3 "" H 6350 4600 50  0001 C CNN
 	1    6350 4600
@@
 	6650 4600 6500 4600
 $Comp
-L R R?
+L R R5
 U 1 1 591C98A4
 P 5500 4350
-F 0 "R?" V 5580 4350 50  0000 C CNN
+F 0 "R5" V 5580 4350 50  0000 C CNN
 F 1 "470" V 5500 4350 50  0000 C CNN
-F 2 "" V 5430 4350 50  0001 C CNN
+F 2 "Resistors_ThroughHole:Resistor_Horizontal_RM10mm" V 5430 4350 50  0001 C CNN
 F 3 "" H 5500 4350 50  0001 C CNN
 	1    5500 4350

Commit message: Massive update of the electrical schematics (Completion of schematics + upgrade to KiCAD 5.0)
Schematics nearly complete, some components references are missing.
The PCB however is still a draft.
Parts:
- added D6: Green, LED_THT:LED_D5.0mm, symbol myrt-rescue:LED-RESCUE-myrt
- added P3: IN, Connector_Phoenix_MC:PhoenixContact_MCV_1,5_2-G-3.5_1x02_P3.50mm_Vertical, symbol myrt-rescue:CONN_2
- added P5: OUT, Connector_PinSocket_2.54mm:PinSocket_1x02_P2.54mm_Vertical, symbol myrt-rescue:CONN_2
- added R10: 500Ω 1% 0.1W, Resistor_THT:R_Axial_Power_L75.0mm_W9.0mm_P86.36mm, symbol myrt-rescue:R
- added R9: 470, Resistor_THT:R_Axial_DIN0204_L3.6mm_D1.6mm_P7.62mm_Horizontal, symbol myrt-rescue:R
- D3, D4, D5: footprint LEDs:LED-5MM -> LED_THT:LED_D5.0mm; symbol LED-RESCUE-myrt -> myrt-rescue:LED-RESCUE-myrt; Manufacturer (none) -> Generic; Vendor (none) -> Stock
- P10, P11, P9: value CONN_2 -> OUT; footprint Connect:bornier2 -> Connector_PinSocket_2.54mm:PinSocket_1x02_P2.54mm_Vertical; symbol CONN_2 -> myrt-rescue:CONN_2; Vendor (none) -> Stock
- P6, P7, P8: value CONN_2 -> IN; footprint Connect:bornier2 -> Connector_Phoenix_MC:PhoenixContact_MCV_1,5_2-G-3.5_1x02_P3.50mm_Vertical; symbol CONN_2 -> myrt-rescue:CONN_2; Vendor (none) -> Stock
- R3, R4, R5: footprint Resistors_ThroughHole:Resistor_Horizontal_RM10mm -> Resistor_THT:R_Axial_DIN0204_L3.6mm_D1.6mm_P7.62mm_Horizontal; symbol R -> myrt-rescue:R; Manufacturer (none) -> Generic; Vendor (none) -> Stock
- R6: value 500Ω 0.1W -> 500Ω 1% 0.1W; footprint Resistors_ThroughHole:Resistor_Horizontal_RM10mm -> Resistor_THT:R_Axial_Power_L75.0mm_W9.0mm_P86.36mm; symbol R -> myrt-rescue:R; Manufacturer (none) -> Multicomp; Order Code (none) -> 2396013; Price (none) -> 0,695€; Product Code (none) -> MCMFR0W4BB5000A50; Vendor (none) -> Farnell; Vendor URL (none) -> https://fr.farnell.com/multicomp/mcmfr0w4bb5000a50/resistan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
- R7: value 100Ω 0.5W -> 100Ω 1% 1W; footprint Resistors_ThroughHole:Resistor_Horizontal_RM30mm -> Resistor_THT:R_Axial_Power_L75.0mm_W9.0mm_P86.36mm; symbol R -> myrt-rescue:R; Manufacturer (none) -> Vishay; Order Code (none) -> 2419015; Price (none) -> 1.42€; Product Code (none) -> CMF70100R00FKEB; Vendor (none) -> Farnell; Vendor URL (none) -> https://fr.farnell.com/vishay/cmf70100r00fkeb/resistance-co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
- R8: value 33Ω 1.5W -> 33Ω 1% 3W; footprint Resistors_ThroughHole:Resistor_Horizontal_RM30mm -> Resistor_THT:R_Axial_Power_L75.0mm_W9.0mm_P86.36mm; symbol R -> myrt-rescue:R; Manufacturer (none) -> Ohmite; Order Code (none) -> 2448938; Price (none) -> 2.16€; Product Code (none) -> 43F33RE; Vendor (none) -> Farnell; Vendor URL (none) -> https://fr.farnell.com/ohmite/43f33re/resis-3w-33-ohm-1-sil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
Connections:
- removed net POWER_5V: P6.1 (P1), P7.1 (P1), P8.1 (P1), R3.2, R4.2, R5.2, R6.2, R7.2, R8.2
- removed net POWER_GND: D3.1 (K), D4.1 (K), D5.1 (K), P10.2 (P2), P11.2 (P2), P6.2 (P2), P7.2 (P2), P8.2 (P2), P9.2 (P2)
- new net: D6.2 (A), R9.1
- new net: P5.1 (P1), R10.1
- new net POWER_5V_S1: P6.1 (P1), R3.2, R6.2
- new net POWER_5V_S2: P7.1 (P1), R4.2, R7.2
- new net POWER_5V_S3: P8.1 (P1), R5.2, R8.2
- new net POWER_5V_S4: P3.1 (P1), R10.2, R9.2
- new net POWER_GND_S1: D3.1 (K), P6.2 (P2), P9.2 (P2)
- new net POWER_GND_S2: D4.1 (K), P10.2 (P2), P7.2 (P2)
- new net POWER_GND_S3: D5.1 (K), P11.2 (P2), P8.2 (P2)
- new net POWER_GND_S4: D6.1 (K), P3.2 (P2), P5.2 (P2)
Other:
- note added: "Accelerated charging station (50mA)"
- note added: "Regular charging station (10mA)"
- note removed: "Medium charging station (50mA)"
- note removed: "Slow charging station (10mA, Two stations)"
- moved on the sheet: D3, D4, D5, P10, P11, P7, P8, P9, R4, R5, R6, R7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

Commit message: PCB creation and update after first prototype built
Parts:
- P3, P6, P7, P8: Manufacturer (none) -> Phoenix Contact; Order Code (none) -> 3704816; Price (none) -> 0,694 €; Product Code (none) -> 1843606; Vendor Stock -> Farnell; Vendor URL (none) -> https://fr.farnell.com/phoenix-contact/1843606/embase-male-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
- R10, R6: footprint Resistor_THT:R_Axial_Power_L75.0mm_W9.0mm_P86.36mm -> Resistor_THT:R_Axial_DIN0207_L6.3mm_D2.5mm_P15.24mm_Horizontal
- R3, R4, R5, R9: footprint Resistor_THT:R_Axial_DIN0204_L3.6mm_D1.6mm_P7.62mm_Horizontal -> Resistor_THT:R_Axial_DIN0207_L6.3mm_D2.5mm_P10.16mm_Horizontal
- R7: footprint Resistor_THT:R_Axial_Power_L75.0mm_W9.0mm_P86.36mm -> Resistor_THT:R_Axial_DIN0516_L15.5mm_D5.0mm_P25.40mm_Horizontal
- R8: footprint Resistor_THT:R_Axial_Power_L75.0mm_W9.0mm_P86.36mm -> Resistor_THT:R_Axial_DIN0614_L14.3mm_D5.7mm_P25.40mm_Horizontal
Changed lines of the file:
@@
 F 2 "Connector_Phoenix_MC:PhoenixContact_MCV_1,5_2-G-3.5_1x02_P3.50mm_Vertical" H 4800 4600 60  0001 C CNN
 F 3 "" H 4800 4600 60  0001 C CNN
-F 4 "Stock" H 0   0   50  0001 C CNN "Vendor"
+F 4 "Farnell" H 0   0   50  0001 C CNN "Vendor"
+F 5 "Phoenix Contact" H 0   0   50  0001 C CNN "Manufacturer"
+F 6 "3704816" H 0   0   50  0001 C CNN "Order Code"
+F 7 "0,694 €" H 0   0   50  0001 C CNN "Price"
+F 8 "1843606" H 0   0   50  0001 C CNN "Product Code"
+F 9 "https://fr.farnell.com/phoenix-contact/1843606/embase-male-verticalee-ci-2v-3/dp/3704816" H 0   0   50  0001 C CNN "Vendor URL"
 	1    4800 4600
 	-1   0    0    -1
@@
 F 0 "R7" V 6930 4500 50  0000 C CNN
 F 1 "100Ω 1% 1W" V 6750 4500 50  0000 C CNN
-F 2 "Resistor_THT:R_Axial_Power_L75.0mm_W9.0mm_P86.36mm" V 6780 4500 50  0001 C CNN
+F 2 "Resistor_THT:R_Axial_DIN0516_L15.5mm_D5.0mm_P25.40mm_Horizontal" V 6780 4500 50  0001 C CNN
 F 3 "" H 6850 4500 50  0001 C CNN
 F 4 "Vishay" H 0   0   50  0001 C CNN "Manufacturer"
@@
 F 0 "R4" V 5580 4250 50  0000 C CNN
 F 1 "470" V 5500 4250 50  0000 C CNN
-F 2 "Resistor_THT:R_Axial_DIN0204_L3.6mm_D1.6mm_P7.62mm_Horizontal" V 5430 4250 50  0001 C CNN
+F 2 "Resistor_THT:R_Axial_DIN0207_L6.3mm_D2.5mm_P10.16mm_Horizontal" V 5430 4250 50  0001 C CNN
 F 3 "" H 5500 4250 50  0001 C CNN
 F 4 "Generic" H 0   0   50  0001 C CNN "Manufacturer"
@@
 F 2 "Connector_Phoenix_MC:PhoenixContact_MCV_1,5_2-G-3.5_1x02_P3.50mm_Vertical" H 4800 2450 60  0001 C CNN
 F 3 "" H 4800 2450 60  0001 C CNN
-F 4 "Stock" H 0   0   50  0001 C CNN "Vendor"
+F 4 "Farnell" H 0   0   50  0001 C CNN "Vendor"
+F 5 "Phoenix Contact" H 0   0   50  0001 C CNN "Manufacturer"
+F 6 "3704816" H 0   0   50  0001 C CNN "Order Code"
+F 7 "0,694 €" H 0   0   50  0001 C CNN "Price"
+F 8 "1843606" H 0   0   50  0001 C CNN "Product Code"
+F 9 "https://fr.farnell.com/phoenix-contact/1843606/embase-male-verticalee-ci-2v-3/dp/3704816" H 0   0   50  0001 C CNN "Vendor URL"
 	1    4800 2450
 	-1   0    0    -1
@@
 F 0 "R6" V 6930 2350 50  0000 C CNN
 F 1 "500Ω 1% 0.1W" V 6750 2350 50  0000 C CNN
-F 2 "Resistor_THT:R_Axial_Power_L75.0mm_W9.0mm_P86.36mm" V 6780 2350 50  0001 C CNN
+F 2 "Resistor_THT:R_Axial_DIN0207_L6.3mm_D2.5mm_P15.24mm_Horizontal" V 6780 2350 50  0001 C CNN
 F 3 "" H 6850 2350 50  0001 C CNN
 F 4 "Multicomp" H 0   0   50  0001 C CNN "Manufacturer"
@@
 F 0 "R3" V 5580 2100 50  0000 C CNN
 F 1 "470" V 5500 2100 50  0000 C CNN
-F 2 "Resistor_THT:R_Axial_DIN0204_L3.6mm_D1.6mm_P7.62mm_Horizontal" V 5430 2100 50  0001 C CNN
+F 2 "Resistor_THT:R_Axial_DIN0207_L6.3mm_D2.5mm_P10.16mm_Horizontal" V 5430 2100 50  0001 C CNN
 F 3 "" H 5500 2100 50  0001 C CNN
 F 4 "Generic" H 0   0   50  0001 C CNN "Manufacturer"
@@
 F 2 "Connector_Phoenix_MC:PhoenixContact_MCV_1,5_2-G-3.5_1x02_P3.50mm_Vertical" H 4800 5700 60  0001 C CNN
 F 3 "" H 4800 5700 60  0001 C CNN
-F 4 "Stock" H 0   0   50  0001 C CNN "Vendor"
+F 4 "Farnell" H 0   0   50  0001 C CNN "Vendor"
+F 5 "Phoenix Contact" H 0   0   50  0001 C CNN "Manufacturer"
+F 6 "3704816" H 0   0   50  0001 C CNN "Order Code"
+F 7 "0,694 €" H 0   0   50  0001 C CNN "Price"
+F 8 "1843606" H 0   0   50  0001 C CNN "Product Code"
+F 9 "https://fr.farnell.com/phoenix-contact/1843606/embase-male-verticalee-ci-2v-3/dp/3704816" H 0   0   50  0001 C CNN "Vendor URL"
 	1    4800 5700
 	-1   0    0    -1
@@
 F 0 "R8" V 6930 5600 50  0000 C CNN
 F 1 "33Ω 1% 3W" V 6750 5600 50  0000 C CNN
-F 2 "Resistor_THT:R_Axial_Power_L75.0mm_W9.0mm_P86.36mm" V 6780 5600 50  0001 C CNN
+F 2 "Resistor_THT:R_Axial_DIN0614_L14.3mm_D5.7mm_P25.40mm_Horizontal" V 6780 5600 50  0001 C CNN
 F 3 "" H 6850 5600 50  0001 C CNN
 F 4 "Ohmite" H 0   0   50  0001 C CNN "Manufacturer"
@@
 F 0 "R5" V 5580 5350 50  0000 C CNN
 F 1 "470" V 5500 5350 50  0000 C CNN
-F 2 "Resistor_THT:R_Axial_DIN0204_L3.6mm_D1.6mm_P7.62mm_Horizontal" V 5430 5350 50  0001 C CNN
+F 2 "Resistor_THT:R_Axial_DIN0207_L6.3mm_D2.5mm_P10.16mm_Horizontal" V 5430 5350 50  0001 C CNN
 F 3 "" H 5500 5350 50  0001 C CNN
 F 4 "Generic" H 0   0   50  0001 C CNN "Manufacturer"
@@
 F 2 "Connector_Phoenix_MC:PhoenixContact_MCV_1,5_2-G-3.5_1x02_P3.50mm_Vertical" H 4800 3500 60  0001 C CNN
 F 3 "" H 4800 3500 60  0001 C CNN
-F 4 "Stock" H 0   0   50  0001 C CNN "Vendor"
+F 4 "Farnell" H 0   0   50  0001 C CNN "Vendor"
+F 5 "Phoenix Contact" H 0   0   50  0001 C CNN "Manufacturer"
+F 6 "3704816" H 0   0   50  0001 C CNN "Order Code"
+F 7 "0,694 €" H 0   0   50  0001 C CNN "Price"
+F 8 "1843606" H 0   0   50  0001 C CNN "Product Code"
+F 9 "https://fr.farnell.com/phoenix-contact/1843606/embase-male-verticalee-ci-2v-3/dp/3704816" H 0   0   50  0001 C CNN "Vendor URL"
 	1    4800 3500
 	-1   0    0    -1
@@
 F 0 "R10" V 6930 3400 50  0000 C CNN
 F 1 "500Ω 1% 0.1W" V 6750 3400 50  0000 C CNN
-F 2 "Resistor_THT:R_Axial_Power_L75.0mm_W9.0mm_P86.36mm" V 6780 3400 50  0001 C CNN
+F 2 "Resistor_THT:R_Axial_DIN0207_L6.3mm_D2.5mm_P15.24mm_Horizontal" V 6780 3400 50  0001 C CNN
 F 3 "" H 6850 3400 50  0001 C CNN
 F 4 "Multicomp" H 0   0   50  0001 C CNN "Manufacturer"
@@
 F 0 "R9" V 5580 3150 50  0000 C CNN
 F 1 "470" V 5500 3150 50  0000 C CNN
-F 2 "Resistor_THT:R_Axial_DIN0204_L3.6mm_D1.6mm_P7.62mm_Horizontal" V 5430 3150 50  0001 C CNN
+F 2 "Resistor_THT:R_Axial_DIN0207_L6.3mm_D2.5mm_P10.16mm_Horizontal" V 5430 3150 50  0001 C CNN
 F 3 "" H 5500 3150 50  0001 C CNN
 F 4 "Generic" H 0   0   50  0001 C CNN "Manufacturer"
