File: src/elec/myrt.sch (KiCad schematic (older format))
At the start: 12 parts

Commit message: Start PCB design
Parts:
- added C1: 10uF, Capacitors_SMD:c_elec_8x10, symbol C
- added D1, D2: 1N4004, Diodes_ThroughHole:Diode_DO-41_SOD81_Horizontal_RM10, symbol D
- added J7: SIL10, Pin_Headers:Pin_Header_Straight_1x10, symbol SIL10
- added P1: Path_Led_Strip, Wire_Connections_Bridges:WireConnection_0.80mmDrill, symbol CONN_2
- added P2: CONN_2, Wire_Connections_Bridges:WireConnection_0.80mmDrill, symbol CONN_2
- added R1: 90, Resistors_ThroughHole:Resistor_Horizontal_RM30mm, symbol R
- added R2: 10, Resistors_ThroughHole:Resistor_Horizontal_RM30mm, symbol R
- C2: renamed from C?; footprint (none) -> Capacitors_ThroughHole:C_Radial_D10_L25_P5
- J1, J2, J3, J4, J5: renamed from J?; footprint (none) -> Connect:USB_A; symbol USB_A -> USB_A-RESCUE-myrt
- J6: renamed from J?; footprint (none) -> Connect:USB_Micro-B; symbol USB_OTG -> USB_OTG-RESCUE-myrt
- P3: renamed from P?; footprint (none) -> Wire_Connections_Bridges:WireConnection_0.80mmDrill
- P4: renamed from P?; value CONN_4 -> HMI_Led_Strip; footprint (none) -> Sockets_MOLEX_KK-System:Socket_MOLEX-KK-RM2-54mm_Lock_4pin_straight
- P5: renamed from P?; footprint (none) -> Connect:bornier2
- U1: renamed from U?; footprint (none) -> Housings_DIP:DIP-18_W7.62mm_LongPads
- U2: renamed from U?; footprint (none) -> Housings_DIP:DIP-32_W15.24mm_LongPads
Connections:
- net labels added: DisplayRx, Vh10, Vharvest
- wire segments 86 -> 107
Other:
- note added: "SW UART on D10"
- note added: "Sparkfun\nSerial 7-Segment Display"
- note added: "To station contacts pads\nfor Energy harvesting measurement"
- note added: "Vh10 Max = 4.8V"
- note added: "Vharvest Max = 48V"
- note added: "White led strip\n(path to Fast Source)"
- moved on the sheet: P4

Commit message: Massive update of the electrical schematics (Completion of schematics + upgrade to KiCAD 5.0)
Schematics nearly complete, some components references are missing.
The PCB however is still a draft.
Parts:
- removed J1, J2, J3, J4, J5: USB_A, Connect:USB_A, symbol USB_A-RESCUE-myrt
- removed J6: USB_OTG, Connect:USB_Micro-B, symbol USB_OTG-RESCUE-myrt
- removed P1: Path_Led_Strip, Wire_Connections_Bridges:WireConnection_0.80mmDrill, symbol CONN_2
- removed P3: RESET_BUT_CON, Wire_Connections_Bridges:WireConnection_0.80mmDrill, symbol CONN_2
- removed P5: START/STOP_BUT_CONN, Connect:bornier2, symbol CONN_2
- removed U1: ULN2803A, Housings_DIP:DIP-18_W7.62mm_LongPads, symbol ULN2803A
- added C3: 100n, Capacitor_THT:C_Rect_L7.0mm_W2.5mm_P5.00mm, symbol Device:C
- added J1: Spare1, Connector_Phoenix_MC:PhoenixContact_MCV_1,5_2-G-3.5_1x02_P3.50mm_Vertical, symbol Connector_Generic:Conn_01x02
- added J10: Spare3, Connector_Phoenix_MC:PhoenixContact_MCV_1,5_2-G-3.5_1x02_P3.50mm_Vertical, symbol Connector_Generic:Conn_01x02
- added J11: Spare4, Connector_Phoenix_MC:PhoenixContact_MCV_1,5_2-G-3.5_1x02_P3.50mm_Vertical, symbol Connector_Generic:Conn_01x02
- added J2: Spare2, Connector_Phoenix_MC:PhoenixContact_MCV_1,5_2-G-3.5_1x02_P3.50mm_Vertical, symbol Connector_Generic:Conn_01x02
- added J3, J4: Regular, Connector_Phoenix_MC:PhoenixContact_MCV_1,5_2-G-3.5_1x02_P3.50mm_Vertical, symbol Connector_Generic:Conn_01x02
- added J6: USB_B PTH Receptable, Connector_USB:USB_B_OST_USB-B1HSxx_Horizontal, symbol Connector:USB_B
- added J8: Accelerated, Connector_Phoenix_MC:PhoenixContact_MCV_1,5_2-G-3.5_1x02_P3.50mm_Vertical, symbol Connector_Generic:Conn_01x02
- added J9: Fast, Connector_Phoenix_MC:PhoenixContact_MCV_1,5_2-G-3.5_1x02_P3.50mm_Vertical, symbol Connector_Generic:Conn_01x02
- added R11: 180Ω 10W, Resistor_THT:R_Axial_Power_L50.0mm_W9.0mm_P55.88mm, symbol myrt-rescue:R
- added R12, R13, R14, R15: 0, Resistor_THT:R_Axial_DIN0204_L3.6mm_D1.6mm_P7.62mm_Horizontal, symbol Device:R
- added SW1: RESET_SW, Button_Switch_THT:SW_PUSH-12mm_Wuerth-430476085716, symbol Switch:SW_Push
- added SW2: START_STOP_SW, Button_Switch_THT:SW_PUSH-12mm_Wuerth-430476085716, symbol Switch:SW_Push
- added U1: ULN2803A, Package_DIP:DIP-18_W7.62mm_Socket_LongPads, symbol Transistor_Array:ULN2803A
- C1: footprint Capacitors_SMD:c_elec_8x10 -> Capacitor_THT:C_Rect_L26.5mm_W8.5mm_P22.50mm_MKS4; symbol C -> myrt-rescue:C; Manufacturer (none) -> Generic; Vendor (none) -> Stock
- C2: value CP -> 100uF; footprint Capacitors_ThroughHole:C_Radial_D10_L25_P5 -> Capacitor_THT:CP_Radial_D10.0mm_P5.00mm; symbol CP -> myrt-rescue:CP; Manufacturer (none) -> Generic; Vendor (none) -> Stock
- D1, D2: footprint Diodes_ThroughHole:Diode_DO-41_SOD81_Horizontal_RM10 -> Diode_THT:D_DO-41_SOD81_P10.16mm_Horizontal; symbol D -> myrt-rescue:D; Manufacturer (none) -> Generic; Vendor (none) -> Stock
- J7: value SIL10 -> Serial 7 Segment Display; footprint Pin_Headers:Pin_Header_Straight_1x10 -> Connector_PinSocket_2.54mm:PinSocket_1x10_P2.54mm_Vertical; symbol SIL10 -> myrt-rescue:SIL10; Manufacturer (none) -> Generic; Note (none) -> Pin row, soldered; Vendor (none) -> Stock
- P2: value CONN_2 -> POWER_DELIVERY; footprint Wire_Connections_Bridges:WireConnection_0.80mmDrill -> Connector_Phoenix_MC:PhoenixContact_MCV_1,5_2-G-3.5_1x02_P3.50mm_Vertical; symbol CONN_2 -> myrt-rescue:CONN_2; Vendor (none) -> Stock
- P4: footprint Sockets_MOLEX_KK-System:Socket_MOLEX-KK-RM2-54mm_Lock_4pin_straight -> Connector_PinSocket_2.54mm:PinSocket_1x04_P2.54mm_Vertical; symbol CONN_4 -> myrt-rescue:CONN_4; Vendor (none) -> Stock
- R1: value 90 -> 180Ω 10W; footprint Resistors_ThroughHole:Resistor_Horizontal_RM30mm -> Resistor_THT:R_Axial_Power_L50.0mm_W9.0mm_P55.88mm; symbol R -> myrt-rescue:R; Manufacturer (none) -> Ohmite; Order Code (none) -> 588-40F180E; Price (none) -> 1.84€; Product Code (none) -> 40F180E; Vendor (none) -> Mouser; Vendor URL (none) -> https://www.mouser.fr/ProductDetail/Ohmite/40F180E?qs=sGAEp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
- R2: value 10 -> 10Ω 3W; footprint Resistors_ThroughHole:Resistor_Horizontal_RM30mm -> Resistor_THT:R_Axial_DIN0516_L15.5mm_D5.0mm_P20.32mm_Horizontal; symbol R -> myrt-rescue:R; Manufacturer (none) -> Vishay; Order Code (none) -> 71-RS02B10R00FE70; Price (none) -> 0.655€; Product Code (none) -> RS02B10R00FE70; Vendor (none) -> Mouser; Vendor URL (none) -> https://www.mouser.fr/ProductDetail/Vishay-Dale/RS02B10R00F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
- U2: footprint Housings_DIP:DIP-32_W15.24mm_LongPads -> Module:Arduino_Nano; symbol arduino-nano-ATmega328 -> myrt-rescue:arduino-nano-ATmega328; Manufacturer (none) -> Arduino; Order Code (none) -> 1848691; Price (none) -> 16.29€; Product Code (none) -> Nano; Vendor (none) -> Farnell; Vendor URL (none) -> https://fr.farnell.com/arduino/a000005/arduino-nano-carte-d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
Connections:
- net labels added: ADC_IN0, RESET_SW, START_SW, SW_UART_DISPLAY
- net labels removed: DisplayRx, RESET_BUT, START/STOP_BUT
- wire segments 107 -> 144
- no-connect marks 5 -> 21
Other:
- note added: "Accelerated\n50mA"
- note added: "Energy delivery input conditionning and protection"
- note added: "Main power supply\nSmartphone charger\n5V/2A output on USB A\nConnect with standard USB A->B Cable"
- note added: "Optionnal limiting resistor\nMount wire if not needed"
- note added: "Regular\n10mA"
- note added: "Sparkfun Serial 7-Segment Display"
- note added: "Vharvest Max = 48V\nReq = 100\nImax = 0.48A\nPmax = 100 * 0.48 * 0.48 = 23W\n\nR 90 : 20W (2x180 10W)\nR 10 : 2.3W"
- note removed: "Fast source\nLed strip"
- note removed: "Main power supply\nSmartphone charger\n5V/2A output on micro-usb"
- note removed: "Medium\n50mA"
- note removed: "SW UART on D10"
- note removed: "Slow\n10mA"
- note removed: "Sparkfun\nSerial 7-Segment Display"
- note removed: "Vharvest Max = 48V"
- note removed: "White led strip\n(path to Fast Source)"
- moved on the sheet: C1, C2, D1, D2, J7, P2, P4, R1, R2, U2

Commit message: PCB creation and update after first prototype built
Parts:
- D1, D2: footprint Diode_THT:D_DO-41_SOD81_P10.16mm_Horizontal -> Diode_THT:D_DO-41_SOD81_P12.70mm_Horizontal
- J1, J10, J11, J2, J4, J8, J9, P2: Manufacturer (none) -> Phoenix Contact; Order Code (none) -> 3704816; Price (none) -> 0,694 €; Product Code (none) -> 1843606; Vendor Stock -> Farnell; Vendor URL (none) -> https://fr.farnell.com/phoenix-contact/1843606/embase-male-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
- J3: Manufacturer (none) -> Phoenix Contact; Notes (none) -> Mate with product 1863152, order code 5089050; Order Code (none) -> 3704816; Price (none) -> 0,694 €; Product Code (none) -> 1843606; Vendor Stock -> Farnell; Vendor URL (none) -> https://fr.farnell.com/phoenix-contact/1843606/embase-male-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
- R1, R11: footprint Resistor_THT:R_Axial_Power_L50.0mm_W9.0mm_P55.88mm -> Resistor_THT:R_Axial_Power_L48.0mm_W12.5mm_P55.88mm
- R12, R13, R14, R15: footprint Resistor_THT:R_Axial_DIN0204_L3.6mm_D1.6mm_P7.62mm_Horizontal -> Resistor_THT:R_Axial_DIN0207_L6.3mm_D2.5mm_P15.24mm_Horizontal
- R2: footprint Resistor_THT:R_Axial_DIN0516_L15.5mm_D5.0mm_P20.32mm_Horizontal -> Resistor_THT:R_Axial_DIN0516_L15.5mm_D5.0mm_P25.40mm_Horizontal
Connections:
- wire segments 144 -> 139
- no-connect marks 21 -> 22
Changed lines of the file:
@@
 	1    0    0    -1
 $EndComp
-Wire Wire Line
-	6200 3050 6300 3050
 Text GLabel 6450 3050 2    60   Input ~ 0
 RESET_SW
@@
 Wire Notes Line
 	3700 4650 2500 4650
-Wire Wire Line
-	4800 3050 4700 3050
-Wire Wire Line
-	4700 3050 4700 2600
-Wire Wire Line
-	4700 2600 6300 2600
-Wire Wire Line
-	6300 2600 6300 3050
-Connection ~ 6300 3050
 $Sheet
 S 9650 6100 1500 300
@@
 F 2 "Connector_Phoenix_MC:PhoenixContact_MCV_1,5_2-G-3.5_1x02_P3.50mm_Vertical" H 950 6650 60  0001 C CNN
 F 3 "" H 950 6650 60  0001 C CNN
-F 4 "Stock" H -3300 1000 50  0001 C CNN "Vendor"
+F 4 "Farnell" H -3300 1000 50  0001 C CNN "Vendor"
+F 5 "Phoenix Contact" H 0   0   50  0001 C CNN "Manufacturer"
+F 6 "3704816" H 0   0   50  0001 C CNN "Order Code"
+F 7 "0,694 €" H 0   0   50  0001 C CNN "Price"
+F 8 "1843606" H 0   0   50  0001 C CNN "Product Code"
+F 9 "https://fr.farnell.com/phoenix-contact/1843606/embase-male-verticalee-ci-2v-3/dp/3704816" H 0   0   50  0001 C CNN "Vendor URL"
 	1    950  6650
 	-1   0    0    1
@@
 F 0 "R1" V 2030 6550 50  0000 C CNN
 F 1 "180Ω 10W" V 1850 6550 50  0000 C CNN
-F 2 "Resistor_THT:R_Axial_Power_L50.0mm_W9.0mm_P55.88mm" V 1880 6550 50  0001 C CNN
+F 2 "Resistor_THT:R_Axial_Power_L48.0mm_W12.5mm_P55.88mm" V 1880 6550 50  0001 C CNN
 F 3 "https://www.mouser.fr/datasheet/2/427/rsns-226497.pdf" H 1950 6550 50  0001 C CNN
 F 4 "Ohmite" H -3300 1000 50  0001 C CNN "Manufacturer"
@@
 F 0 "R2" V 2280 6750 50  0000 C CNN
 F 1 "10Ω 3W" V 2100 6750 50  0000 C CNN
-F 2 "Resistor_THT:R_Axial_DIN0516_L15.5mm_D5.0mm_P20.32mm_Horizontal" V 2130 6750 50  0001 C CNN
+F 2 "Resistor_THT:R_Axial_DIN0516_L15.5mm_D5.0mm_P25.40mm_Horizontal" V 2130 6750 50  0001 C CNN
 F 3 "https://www.mouser.fr/datasheet/2/427/rsns-226497.pdf" H 2200 6750 50  0001 C CNN
 F 4 "Vishay" H 2200 6750 50  0001 C CNN "Manufacturer"
@@
 F 0 "D1" H 3300 6450 50  0000 C CNN
 F 1 "1N4004" H 3300 6250 50  0000 C CNN
-F 2 "Diode_THT:D_DO-41_SOD81_P10.16mm_Horizontal" H 3300 6350 50  0001 C CNN
+F 2 "Diode_THT:D_DO-41_SOD81_P12.70mm_Horizontal" H 3300 6350 50  0001 C CNN
 F 3 "" H 3300 6350 50  0000 C CNN
 F 4 "Generic" H 3300 6350 50  0001 C CNN "Manufacturer"
@@
 F 0 "D2" H 3300 6850 50  0000 C CNN
 F 1 "1N4004" H 3300 6650 50  0000 C CNN
-F 2 "Diode_THT:D_DO-41_SOD81_P10.16mm_Horizontal" H 3300 6750 50  0001 C CNN
+F 2 "Diode_THT:D_DO-41_SOD81_P12.70mm_Horizontal" H 3300 6750 50  0001 C CNN
 F 3 "" H 3300 6750 50  0000 C CNN
 F 4 "Generic" H 3300 6750 50  0001 C CNN "Manufacturer"
@@
 Wire Wire Line
 	5950 1350 5950 1500
-Wire Wire Line
-	6300 3050 6450 3050
 Wire Wire Line
 	2200 6900 2500 6900
@@
 F 0 "R11" V 2030 6250 50  0000 C CNN
 F 1 "180Ω 10W" V 1850 6250 50  0000 C CNN
-F 2 "Resistor_THT:R_Axial_Power_L50.0mm_W9.0mm_P55.88mm" V 1880 6250 50  0001 C CNN
+F 2 "Resistor_THT:R_Axial_Power_L48.0mm_W12.5mm_P55.88mm" V 1880 6250 50  0001 C CNN
 F 3 "https://www.mouser.fr/datasheet/2/427/rsns-226497.pdf" H 1950 6250 50  0001 C CNN
 F 4 "Ohmite" H 1950 6250 50  0001 C CNN "Manufacturer"
@@
 F 0 "R12" V 1443 3750 50  0000 C CNN
 F 1 "0" V 1534 3750 50  0000 C CNN
-F 2 "Resistor_THT:R_Axial_DIN0204_L3.6mm_D1.6mm_P7.62mm_Horizontal" V 1580 3750 50  0001 C CNN
+F 2 "Resistor_THT:R_Axial_DIN0207_L6.3mm_D2.5mm_P15.24mm_Horizontal" V 1580 3750 50  0001 C CNN
 F 3 "~" H 1650 3750 50  0001 C CNN
 F 4 "Stock" H -300 -2450 50  0001 C CNN "Vendor"
@@
 F 2 "Connector_Phoenix_MC:PhoenixContact_MCV_1,5_2-G-3.5_1x02_P3.50mm_Vertical" H 1300 1200 50  0001 C CNN
 F 3 "~" H 1300 1200 50  0001 C CNN
-F 4 "Stock" H 0   0   50  0001 C CNN "Vendor"
+F 4 "Phoenix Contact" H 0   0   50  0001 C CNN "Manufacturer"
+F 5 "1843606" H 0   0   50  0001 C CNN "Product Code"
+F 6 "Farnell" H 0   0   50  0001 C CNN "Vendor"
+F 7 "3704816" H 0   0   50  0001 C CNN "Order Code"
+F 8 "https://fr.farnell.com/phoenix-contact/1843606/embase-male-verticalee-ci-2v-3/dp/3704816" H 0   0   50  0001 C CNN "Vendor URL"
+F 9 "0,694 €" H 0   0   50  0001 C CNN "Price"
+F 10 "Mate with product 1863152, order code 5089050" H 1300 1200 50  0001 C CNN "Notes"
 	1    1300 1200
 	-1   0    0    -1
@@
 F 2 "Connector_Phoenix_MC:PhoenixContact_MCV_1,5_2-G-3.5_1x02_P3.50mm_Vertical" H 1300 1750 50  0001 C CNN
 F 3 "~" H 1300 1750 50  0001 C CNN
-F 4 "Stock" H 0   0   50  0001 C CNN "Vendor"
+F 4 "Farnell" H 0   0   50  0001 C CNN "Vendor"
+F 5 "Phoenix Contact" H 0   0   50  0001 C CNN "Manufacturer"
+F 6 "3704816" H 0   0   50  0001 C CNN "Order Code"
+F 7 "0,694 €" H 0   0   50  0001 C CNN "Price"
+F 8 "1843606" H 0   0   50  0001 C CNN "Product Code"
+F 9 "https://fr.farnell.com/phoenix-contact/1843606/embase-male-verticalee-ci-2v-3/dp/3704816" H 0   0   50  0001 C CNN "Vendor URL"
 	1    1300 1750
 	-1   0    0    -1
@@
 F 2 "Connector_Phoenix_MC:PhoenixContact_MCV_1,5_2-G-3.5_1x02_P3.50mm_Vertical" H 1300 2300 50  0001 C CNN
 F 3 "~" H 1300 2300 50  0001 C CNN
-F 4 "Stock" H 0   0   50  0001 C CNN "Vendor"
+F 4 "Farnell" H 0   0   50  0001 C CNN "Vendor"
+F 5 "Phoenix Contact" H 0   0   50  0001 C CNN "Manufacturer"
+F 6 "3704816" H 0   0   50  0001 C CNN "Order Code"
+F 7 "0,694 €" H 0   0   50  0001 C CNN "Price"
+F 8 "1843606" H 0   0   50  0001 C CNN "Product Code"
+F 9 "https://fr.farnell.com/phoenix-contact/1843606/embase-male-verticalee-ci-2v-3/dp/3704816" H 0   0   50  0001 C CNN "Vendor URL"
 	1    1300 2300
 	-1   0    0    -1
@@
 F 2 "Connector_Phoenix_MC:PhoenixContact_MCV_1,5_2-G-3.5_1x02_P3.50mm_Vertical" H 1300 2850 50  0001 C CNN
 F 3 "~" H 1300 2850 50  0001 C CNN
-F 4 "Stock" H 0   0   50  0001 C CNN "Vendor"
+F 4 "Farnell" H 0   0   50  0001 C CNN "Vendor"
+F 5 "Phoenix Contact" H 0   0   50  0001 C CNN "Manufacturer"
+F 6 "3704816" H 0   0   50  0001 C CNN "Order Code"
+F 7 "0,694 €" H 0   0   50  0001 C CNN "Price"
+F 8 "1843606" H 0   0   50  0001 C CNN "Product Code"
+F 9 "https://fr.farnell.com/phoenix-contact/1843606/embase-male-verticalee-ci-2v-3/dp/3704816" H 0   0   50  0001 C CNN "Vendor URL"
 	1    1300 2850
 	-1   0    0    -1
@@
 F 2 "Connector_Phoenix_MC:PhoenixContact_MCV_1,5_2-G-3.5_1x02_P3.50mm_Vertical" H 900 3800 50  0001 C CNN
 F 3 "~" H 900 3800 50  0001 C CNN
-F 4 "Stock" H 900 3800 50  0001 C CNN "Vendor"
+F 4 "Farnell" H 900 3800 50  0001 C CNN "Vendor"
+F 5 "Phoenix Contact" H 0   0   50  0001 C CNN "Manufacturer"
+F 6 "3704816" H 0   0   50  0001 C CNN "Order Code"
+F 7 "0,694 €" H 0   0   50  0001 C CNN "Price"
+F 8 "1843606" H 0   0   50  0001 C CNN "Product Code"
+F 9 "https://fr.farnell.com/phoenix-contact/1843606/embase-male-verticalee-ci-2v-3/dp/3704816" H 0   0   50  0001 C CNN "Vendor URL"
 	1    900  3800
 	-1   0    0    -1
@@
 F 2 "Connector_Phoenix_MC:PhoenixContact_MCV_1,5_2-G-3.5_1x02_P3.50mm_Vertical" H 900 4300 50  0001 C CNN
 F 3 "~" H 900 4300 50  0001 C CNN
-F 4 "Stock" H 900 4300 50  0001 C CNN "Vendor"
+F 4 "Farnell" H 900 4300 50  0001 C CNN "Vendor"
+F 5 "Phoenix Contact" H 0   0   50  0001 C CNN "Manufacturer"
+F 6 "3704816" H 0   0   50  0001 C CNN "Order Code"
+F 7 "0,694 €" H 0   0   50  0001 C CNN "Price"
+F 8 "1843606" H 0   0   50  0001 C CNN "Product Code"
+F 9 "https://fr.farnell.com/phoenix-contact/1843606/embase-male-verticalee-ci-2v-3/dp/3704816" H 0   0   50  0001 C CNN "Vendor URL"
 	1    900  4300
 	-1   0    0    -1
@@
 F 0 "R13" V 1443 4300 50  0000 C CNN
 F 1 "0" V 1534 4300 50  0000 C CNN
-F 2 "Resistor_THT:R_Axial_DIN0204_L3.6mm_D1.6mm_P7.62mm_Horizontal" V 1580 4300 50  0001 C CNN
+F 2 "Resistor_THT:R_Axial_DIN0207_L6.3mm_D2.5mm_P15.24mm_Horizontal" V 1580 4300 50  0001 C CNN
 F 3 "~" H 1650 4300 50  0001 C CNN
 F 4 "Stock" H -300 -1900 50  0001 C CNN "Vendor"
@@
 F 0 "R14" V 1443 4750 50  0000 C CNN
 F 1 "0" V 1534 4750 50  0000 C CNN
-F 2 "Resistor_THT:R_Axial_DIN0204_L3.6mm_D1.6mm_P7.62mm_Horizontal" V 1580 4750 50  0001 C CNN
+F 2 "Resistor_THT:R_Axial_DIN0207_L6.3mm_D2.5mm_P15.24mm_Horizontal" V 1580 4750 50  0001 C CNN
 F 3 "~" H 1650 4750 50  0001 C CNN
 F 4 "Stock" H -300 -1450 50  0001 C CNN "Vendor"
@@
 F 2 "Connector_Phoenix_MC:PhoenixContact_MCV_1,5_2-G-3.5_1x02_P3.50mm_Vertical" H 900 4800 50  0001 C CNN
 F 3 "~" H 900 4800 50  0001 C CNN
-F 4 "Stock" H 0   0   50  0001 C CNN "Vendor"
+F 4 "Farnell" H 0   0   50  0001 C CNN "Vendor"
+F 5 "Phoenix Contact" H 0   0   50  0001 C CNN "Manufacturer"
+F 6 "3704816" H 0   0   50  0001 C CNN "Order Code"
+F 7 "0,694 €" H 0   0   50  0001 C CNN "Price"
+F 8 "1843606" H 0   0   50  0001 C CNN "Product Code"
+F 9 "https://fr.farnell.com/phoenix-contact/1843606/embase-male-verticalee-ci-2v-3/dp/3704816" H 0   0   50  0001 C CNN "Vendor URL"
 	1    900  4800
 	-1   0    0    -1
@@
 F 0 "R15" V 1443 5250 50  0000 C CNN
 F 1 "0" V 1534 5250 50  0000 C CNN
-F 2 "Resistor_THT:R_Axial_DIN0204_L3.6mm_D1.6mm_P7.62mm_Horizontal" V 1580 5250 50  0001 C CNN
+F 2 "Resistor_THT:R_Axial_DIN0207_L6.3mm_D2.5mm_P15.24mm_Horizontal" V 1580 5250 50  0001 C CNN
 F 3 "~" H 1650 5250 50  0001 C CNN
 F 4 "Stock" H -300 -950 50  0001 C CNN "Vendor"
@@
 F 2 "Connector_Phoenix_MC:PhoenixContact_MCV_1,5_2-G-3.5_1x02_P3.50mm_Vertical" H 900 5300 50  0001 C CNN
 F 3 "~" H 900 5300 50  0001 C CNN
-F 4 "Stock" H 0   0   50  0001 C CNN "Vendor"
+F 4 "Farnell" H 0   0   50  0001 C CNN "Vendor"
+F 5 "Phoenix Contact" H 0   0   50  0001 C CNN "Manufacturer"
+F 6 "3704816" H 0   0   50  0001 C CNN "Order Code"
+F 7 "0,694 €" H 0   0   50  0001 C CNN "Price"
+F 8 "1843606" H 0   0   50  0001 C CNN "Product Code"
+F 9 "https://fr.farnell.com/phoenix-contact/1843606/embase-male-verticalee-ci-2v-3/dp/3704816" H 0   0   50  0001 C CNN "Vendor URL"
 	1    900  5300
 	-1   0    0    -1
@@
 Wire Notes Line
 	8300 5250 8300 1800
+Wire Wire Line
+	6200 3050 6450 3050
+NoConn ~ 4800 3050
 $EndSCHEMATC

Commit message: Deleted useless component (C), minor changes after tests
Parts:
- removed C1: 10uF, Capacitor_THT:C_Rect_L26.5mm_W8.5mm_P22.50mm_MKS4, symbol myrt-rescue:C
Connections:
- wire segments 139 -> 136
Changed lines of the file:
@@
 	1450 6750 1300 6750
 Connection ~ 2200 6550
-$Comp
-L myrt-rescue:C C1
-U 1 1 5B461EE5
-P 2500 6700
-F 0 "C1" H 2525 6800 50  0000 L CNN
-F 1 "10uF" H 2525 6600 50  0000 L CNN
-F 2 "Capacitor_THT:C_Rect_L26.5mm_W8.5mm_P22.50mm_MKS4" H 2538 6550 50  0001 C CNN
-F 3 "" H 2500 6700 50  0000 C CNN
-F 4 "No polarity" H 2500 6700 60  0001 C CNN "Note"
-F 5 "Generic" H -3300 1000 50  0001 C CNN "Manufacturer"
-F 6 "Stock" H -3300 1000 50  0001 C CNN "Vendor"
-	1    2500 6700
-	1    0    0    -1
-$EndComp
-Wire Wire Line
-	2500 6900 2500 6850
 Connection ~ 2200 6900
 $Comp
@@
 	3300 6500 3300 6550
 Connection ~ 3300 6550
-Connection ~ 2500 6900
 $Comp
 L power:+5V #PWR021
@@
 Wire Wire Line
 	5950 1350 5950 1500
-Wire Wire Line
-	2200 6900 2500 6900
 Wire Wire Line
 	3300 6550 3300 6600
@@
 Wire Wire Line
 	2150 6550 2200 6550
-Connection ~ 2500 6550
-Wire Wire Line
-	2200 6550 2500 6550
-Wire Wire Line
-	2500 6900 3300 6900
-Wire Wire Line
-	2500 6550 3300 6550
 $Comp
 L Device:R R12
@@
 	6200 3050 6450 3050
 NoConn ~ 4800 3050
+Wire Wire Line
+	2200 6550 3300 6550
+Wire Wire Line
+	2200 6900 3300 6900
 $EndSCHEMATC
