File: src/elec/myrt.kicad_pcb (KiCad board)
At the start: 2 copper layers, 0 parts

Commit message: Start PCB design
Parts:
- added C1: 10uF, Capacitors_SMD:c_elec_8x10, F.Cu at (128.3, 85.1)
- added C2: CP, Capacitors_ThroughHole:C_Radial_D10_L25_P5, F.Cu at (119.4, 121.9)
- added D1: 1N4004, Diodes_ThroughHole:Diode_DO-41_SOD81_Horizontal_RM10, F.Cu at (118.1, 74.9)
- added D2: 1N4004, Diodes_ThroughHole:Diode_DO-41_SOD81_Horizontal_RM10, F.Cu at (104.1, 77.5)
- added D3: Green, LEDs:LED-5MM, F.Cu at (91.4, 120.7)
- added D4: Yellow, LEDs:LED-5MM, F.Cu at (83.8, 120.7)
- added D5: Red, LEDs:LED-5MM, F.Cu at (99.1, 120.7)
- added J1: USB_A, Connect:USB_A, F.Cu at (113.0, 167.6)
- added J2: USB_A, Connect:USB_A, F.Cu at (113.0, 149.9)
- added J3: USB_A, Connect:USB_A, F.Cu at (115.6, 132.1)
- added J4: USB_A, Connect:USB_A, F.Cu at (95.2, 153.7)
- added J5: USB_A, Connect:USB_A, F.Cu at (95.2, 170.2)
- added J6: USB_OTG, Connect:USB_Micro-B, F.Cu at (116.8, 86.4)
- added J7: SIL10, Pin_Headers:Pin_Header_Straight_1x10, F.Cu at (132.1, 120.7)
- added P1: Path_Led_Strip, Wire_Connections_Bridges:WireConnection_0.80mmDrill, F.Cu at (92.7, 147.3)
- added P10: CONN_2, Connect:bornier2, F.Cu at (110.5, 120.7)
- added P11: CONN_2, Connect:bornier2, F.Cu at (104.1, 132.1)
- added P2: CONN_2, Wire_Connections_Bridges:WireConnection_0.80mmDrill, F.Cu at (151.1, 102.9)
- added P3: RESET_BUT_CON, Wire_Connections_Bridges:WireConnection_0.80mmDrill, F.Cu at (132.1, 104.1)
- added P4: HMI_Led_Strip, Sockets_MOLEX_KK-System:Socket_MOLEX-KK-RM2-54mm_Lock_4pin_straight, F.Cu at (133.3, 180.3)
- added P5: START/STOP_BUT_CONN, Connect:bornier2, F.Cu at (105.4, 86.4)
- added P6: CONN_2, Connect:bornier2, F.Cu at (121.9, 109.2)
- added P7: CONN_2, Connect:bornier2, F.Cu at (121.9, 97.8)
- added P8: CONN_2, Connect:bornier2, F.Cu at (110.5, 109.2)
- added P9: CONN_2, Connect:bornier2, F.Cu at (110.5, 97.8)
- added R1: 90, Resistors_ThroughHole:Resistor_Horizontal_RM30mm, F.Cu at (135.9, 73.7)
- added R2: 10, Resistors_ThroughHole:Resistor_Horizontal_RM30mm, F.Cu at (135.9, 87.6)
- added R3: 470, Resistors_ThroughHole:Resistor_Horizontal_RM10mm, F.Cu at (86.4, 135.9)
- added R4: 470, Resistors_ThroughHole:Resistor_Horizontal_RM10mm, F.Cu at (86.4, 128.3)
- added R5: 470, Resistors_ThroughHole:Resistor_Horizontal_RM10mm, F.Cu at (92.7, 110.5)
- added R6: 500Ω 0.1W, Resistors_ThroughHole:Resistor_Horizontal_RM10mm, F.Cu at (92.7, 100.3)
- added R7: 100Ω 0.5W, Resistors_ThroughHole:Resistor_Horizontal_RM30mm, F.Cu at (135.9, 114.3)
- added R8: 33Ω 1.5W, Resistors_ThroughHole:Resistor_Horizontal_RM30mm, F.Cu at (135.9, 128.3)
- added U1: ULN2803A, Housings_DIP:DIP-18_W7.62mm_LongPads, F.Cu at (129.5, 152.4)
- added U2: arduino-nano-ATmega328, Housings_DIP:DIP-32_W15.24mm_LongPads, F.Cu at (149.9, 143.5)
Other:
- board outline added: 113 x 132.1 mm

Commit message: Massive update of the electrical schematics (Completion of schematics + upgrade to KiCAD 5.0)
Schematics nearly complete, some components references are missing.
The PCB however is still a draft.
Parts:
- removed J5: USB_A, Connect:USB_A
- added C3: 100n, Capacitor_THT:C_Rect_L7.0mm_W2.5mm_P5.00mm, F.Cu at (63.5, 76.2)
- added D6: Green, LED_THT:LED_D5.0mm, F.Cu at (250.4, 255.6)
- added P12: Path_Led_Strip, Connector_Wire:SolderWirePad_1x02_P5.08mm_Drill1.5mm, F.Cu at (74.3, 165.5)
- added R10: 500Ω 0.1W, Resistor_THT:R_Axial_DIN0204_L3.6mm_D1.6mm_P7.62mm_Horizontal, F.Cu at (239.7, 260.4)
- added R11: 180Ω 10W, Resistor_THT:R_Axial_Power_L50.0mm_W9.0mm_P55.88mm, F.Cu at (58.6, 158.4)
- added R12: R, Resistor_THT:R_Axial_DIN0309_L9.0mm_D3.2mm_P12.70mm_Horizontal, F.Cu at (58.2, 165.1)
- added R9: 470, Resistor_THT:R_Axial_DIN0204_L3.6mm_D1.6mm_P7.62mm_Horizontal, F.Cu at (249.4, 251.3)
- added SW1: RESET_SW, Button_Switch_THT:SW_PUSH-12mm_Wuerth-430476085716, F.Cu at (29.2, 53.3)
- added SW2: START_STOP_SW, Button_Switch_THT:SW_PUSH-12mm_Wuerth-430476085716, F.Cu at (121.9, 53.3)
- C1: footprint Capacitors_SMD:c_elec_8x10 -> Capacitor_THT:C_Rect_L26.5mm_W8.5mm_P22.50mm_MKS4
- C2: footprint Capacitors_ThroughHole:C_Radial_D10_L25_P5 -> Capacitor_THT:CP_Radial_D10.0mm_P5.00mm
- D1, D2: footprint Diodes_ThroughHole:Diode_DO-41_SOD81_Horizontal_RM10 -> Diode_THT:D_DO-41_SOD81_P10.16mm_Horizontal
- D3, D4, D5: footprint LEDs:LED-5MM -> LED_THT:LED_D5.0mm
- J1, J2: value USB_A -> Regular; footprint Connect:USB_A -> Connector_USB:USB3_A_Molex_48393-001
- J3: value USB_A -> Accelerated; footprint Connect:USB_A -> Connector_USB:USB3_A_Molex_48393-001
- J4: value USB_A -> Fast; footprint Connect:USB_A -> Connector_USB:USB3_A_Molex_48393-001
- J6: footprint Connect:USB_Micro-B -> Connector_USB:USB_Micro-B_Wuerth_629105150521_CircularHoles; moved to B.Cu
- J7: footprint Pin_Headers:Pin_Header_Straight_1x10 -> Connector_PinSocket_2.54mm:PinSocket_1x10_P2.54mm_Vertical
- P1, P2: footprint Wire_Connections_Bridges:WireConnection_0.80mmDrill -> Connector_Wire:SolderWirePad_1x02_P5.08mm_Drill1.5mm
- P10, P11, P9: value CONN_2 -> OUT; footprint Connect:bornier2 -> Connector_Wire:SolderWirePad_1x02_P5.08mm_Drill1.5mm
- P3: value RESET_BUT_CON -> IN; footprint Wire_Connections_Bridges:WireConnection_0.80mmDrill -> Connector_Wire:SolderWirePad_1x02_P5.08mm_Drill1.5mm
- P4: footprint Sockets_MOLEX_KK-System:Socket_MOLEX-KK-RM2-54mm_Lock_4pin_straight -> Connector_Wire:SolderWirePad_1x04_P3.81mm_Drill1mm
- P5: value START/STOP_BUT_CONN -> OUT; footprint Connect:bornier2 -> Connector_Wire:SolderWirePad_1x02_P5.08mm_Drill1.5mm
- P6, P7, P8: value CONN_2 -> IN; footprint Connect:bornier2 -> Connector_Wire:SolderWirePad_1x02_P5.08mm_Drill1.5mm
- R1: value 90 -> 180Ω 10W; footprint Resistors_ThroughHole:Resistor_Horizontal_RM30mm -> Resistor_THT:R_Axial_Power_L50.0mm_W9.0mm_P55.88mm
- R2: value 10 -> 10Ω 3W; footprint Resistors_ThroughHole:Resistor_Horizontal_RM30mm -> Resistor_THT:R_Axial_Power_L50.0mm_W9.0mm_P55.88mm
- R3, R4, R5, R6: footprint Resistors_ThroughHole:Resistor_Horizontal_RM10mm -> Resistor_THT:R_Axial_DIN0204_L3.6mm_D1.6mm_P7.62mm_Horizontal
- R7, R8: footprint Resistors_ThroughHole:Resistor_Horizontal_RM30mm -> Resistor_THT:R_Axial_Power_L50.0mm_W9.0mm_P55.88mm
- U1: footprint Housings_DIP:DIP-18_W7.62mm_LongPads -> Package_DIP:DIP-18_W7.62mm_Socket_LongPads
- U2: footprint Housings_DIP:DIP-32_W15.24mm_LongPads -> Module:Arduino_Nano
- moved R6 223.0 mm to (279.4, 222.2), turned to 180 degrees
- moved P5 218.0 mm to (241.0, 257.0)
- moved R3 217.1 mm to (283.2, 227.3)
- moved D3 214.6 mm to (273.1, 234.9)
- moved P3 184.0 mm to (241.0, 252.5)
- moved P6 181.4 mm to (247.7, 240.0)
- moved R5 174.5 mm to (251.5, 38.1)
- moved P9 166.8 mm to (217.2, 226.1)
- moved D5 166.7 mm to (243.8, 38.1)
- moved R4 163.9 mm to (241.3, 181.6)
- moved D4 152.2 mm to (227.3, 171.4)
- moved R8 136.8 mm to (238.8, 38.1), turned to 180 degrees
- moved P10 133.8 mm to (238.8, 158.8), turned to 90 degrees
- moved P7 119.1 mm to (223.5, 160.0)
- moved P4 117.3 mm to (113.0, 64.8)
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Connections:
- D3 pad 1: /Charging stations/POWER_GND -> /Charging stations/POWER_GND_S1
- D4 pad 1: /Charging stations/POWER_GND -> /Charging stations/POWER_GND_S2
- D5 pad 1: /Charging stations/POWER_GND -> /Charging stations/POWER_GND_S3
- J1 pad 2: Net-(J1-Pad2) -> (no net)
- J1 pad 3: Net-(J1-Pad3) -> (no net)
- J2 pad 2: Net-(J2-Pad2) -> (no net)
- J2 pad 3: Net-(J2-Pad3) -> (no net)
- J3 pad 2: Net-(J3-Pad2) -> (no net)
- J3 pad 3: Net-(J3-Pad3) -> (no net)
- J4 pad 2: Net-(J4-Pad2) -> (no net)
- J4 pad 3: Net-(J4-Pad3) -> (no net)
- J6 pad 2: Net-(J6-Pad2) -> (no net)
- J6 pad 3: Net-(J6-Pad3) -> (no net)
- J6 pad 4: Net-(J6-Pad4) -> (no net)
- J7 pad 10: Net-(J7-Pad10) -> (no net)
- J7 pad 2: Net-(J7-Pad2) -> (no net)
- J7 pad 3: Net-(J7-Pad3) -> (no net)
- J7 pad 4: Net-(J7-Pad4) -> (no net)
- J7 pad 5: Net-(J7-Pad5) -> (no net)
- J7 pad 6: Net-(J7-Pad6) -> (no net)
- J7 pad 9: Net-(J7-Pad9) -> (no net)
- P10 pad 2: /Charging stations/POWER_GND -> /Charging stations/POWER_GND_S2
- P11 pad 2: /Charging stations/POWER_GND -> /Charging stations/POWER_GND_S3
- P3 pad 1: RESET_BUT -> /Charging stations/POWER_5V_S4
- P3 pad 2: GND -> /Charging stations/POWER_GND_S4
- P5 pad 1: START/STOP_BUT -> Net-(P5-Pad1)
- P5 pad 2: GND -> /Charging stations/POWER_GND_S4
- P6 pad 1: /Charging stations/POWER_5V -> /Charging stations/POWER_5V_S1
- P6 pad 2: /Charging stations/POWER_GND -> /Charging stations/POWER_GND_S1
- P7 pad 1: /Charging stations/POWER_5V -> /Charging stations/POWER_5V_S2
- P7 pad 2: /Charging stations/POWER_GND -> /Charging stations/POWER_GND_S2
- P8 pad 1: /Charging stations/POWER_5V -> /Charging stations/POWER_5V_S3
- P8 pad 2: /Charging stations/POWER_GND -> /Charging stations/POWER_GND_S3
- P9 pad 2: /Charging stations/POWER_GND -> /Charging stations/POWER_GND_S1
- R3 pad 2: /Charging stations/POWER_5V -> /Charging stations/POWER_5V_S1
- R4 pad 2: /Charging stations/POWER_5V -> /Charging stations/POWER_5V_S2
- R5 pad 2: /Charging stations/POWER_5V -> /Charging stations/POWER_5V_S3
- R6 pad 2: /Charging stations/POWER_5V -> /Charging stations/POWER_5V_S1
- R7 pad 2: /Charging stations/POWER_5V -> /Charging stations/POWER_5V_S2
- R8 pad 2: /Charging stations/POWER_5V -> /Charging stations/POWER_5V_S3
- U1 pad 1: Net-(J1-Pad4) -> GND
- U1 pad 11: Net-(U1-Pad11) -> Net-(J1-Pad4)
- U1 pad 12: Net-(U1-Pad12) -> Net-(J2-Pad4)
- U1 pad 13: Net-(U1-Pad13) -> Net-(J3-Pad4)
- U1 pad 14: Net-(U1-Pad14) -> Net-(J4-Pad4)
- U1 pad 15: Net-(U1-Pad15) -> Net-(P12-Pad2)
- U1 pad 16: Net-(U1-Pad16) -> Net-(P1-Pad2)
- U1 pad 17: Net-(U1-Pad17) -> (no net)
- U1 pad 18: Net-(U1-Pad18) -> (no net)
- U1 pad 2: Net-(J2-Pad4) -> GND
- U1 pad 3: Net-(J3-Pad4) -> Net-(U1-Pad3)
- U1 pad 4: Net-(J4-Pad4) -> Net-(U1-Pad4)
- U1 pad 5: Net-(J5-Pad4) -> Net-(U1-Pad5)
- U1 pad 7: Net-(P1-Pad2) -> Net-(U1-Pad7)
- U2 pad 1: Net-(U2-Pad1) -> (no net)
- U2 pad 10: Net-(U1-Pad12) -> Net-(U1-Pad4)
- U2 pad 11: Net-(U2-Pad11) -> Net-(U1-Pad3)
- U2 pad 12: Net-(U2-Pad12) -> (no net)
- U2 pad 15: Net-(U2-Pad15) -> (no net)
- U2 pad 17: Net-(U2-Pad17) -> (no net)
- U2 pad 18: Net-(U2-Pad18) -> (no net)
- U2 pad 2: Net-(U2-Pad2) -> (no net)
- U2 pad 20: Net-(U2-Pad20) -> (no net)
- U2 pad 21: Net-(U2-Pad21) -> (no net)
- U2 pad 22: Net-(U2-Pad22) -> (no net)
- U2 pad 23: Net-(U2-Pad23) -> (no net)
- U2 pad 24: Net-(U2-Pad24) -> (no net)
- U2 pad 25: Net-(U2-Pad25) -> (no net)
- U2 pad 26: Net-(U2-Pad26) -> (no net)
- U2 pad 28: RESET_BUT -> RESET_SW
- U2 pad 3: RESET_BUT -> RESET_SW
- U2 pad 30: Net-(U2-Pad30) -> (no net)
- U2 pad 5: Net-(U1-Pad18) -> START_SW
- U2 pad 6: Net-(U1-Pad17) -> Net-(U1-Pad8)
- U2 pad 7: Net-(U1-Pad16) -> Net-(U1-Pad7)
- U2 pad 8: Net-(U1-Pad15) -> Net-(U1-Pad6)
- U2 pad 9: Net-(U1-Pad14) -> Net-(U1-Pad5)
Other:
- board size 113 x 132.1 mm -> 259.1 x 109.2 mm
- board text added: "Energy Storage Station PVC Tube, 20cm height, 10cm diameter (9.2 inner)"
- board text added: "Fast source"
- board text added: "RESET"
- board text added: "START"
- board text added: "Sources PVC Tube, 20cm height, 8cm diameter (7.2 inner)"

Commit message: PCB creation and update after first prototype built
Parts:
- removed P1, P12: Path_Led_Strip, Connector_Wire:SolderWirePad_1x02_P5.08mm_Drill1.5mm
- added J10: Spare3, Connector_Phoenix_MC:PhoenixContact_MCV_1,5_2-G-3.5_1x02_P3.50mm_Vertical, F.Cu at (112.5, 82.2)
- added J11: Spare4, Connector_Phoenix_MC:PhoenixContact_MCV_1,5_2-G-3.5_1x02_P3.50mm_Vertical, F.Cu at (96.3, 82.2)
- added J8: Accelerated, Connector_Phoenix_MC:PhoenixContact_MCV_1,5_2-G-3.5_1x02_P3.50mm_Vertical, F.Cu at (64.8, 82.9)
- added J9: Fast, Connector_Phoenix_MC:PhoenixContact_MCV_1,5_2-G-3.5_1x02_P3.50mm_Vertical, F.Cu at (64.8, 72.8)
- added R13: 0, Resistor_THT:R_Axial_DIN0207_L6.3mm_D2.5mm_P15.24mm_Horizontal, F.Cu at (119.4, 98.2)
- added R14: 0, Resistor_THT:R_Axial_DIN0207_L6.3mm_D2.5mm_P15.24mm_Horizontal, F.Cu at (106.2, 99.2)
- added R15: 0, Resistor_THT:R_Axial_DIN0207_L6.3mm_D2.5mm_P15.24mm_Horizontal, F.Cu at (102.9, 99.2)
- added REF**: MountingHole_3.2mm_M3_ISO7380_Pad, MountingHole:MountingHole_3.2mm_M3_ISO7380_Pad, F.Cu at (136.1, 177.2)
- added REF**: MountingHole_3.2mm_M3_ISO7380_Pad, MountingHole:MountingHole_3.2mm_M3_ISO7380_Pad, F.Cu at (136.0, 202.9)
- added REF**: MountingHole_3.2mm_M3_ISO7380_Pad, MountingHole:MountingHole_3.2mm_M3_ISO7380_Pad, F.Cu at (68.7, 229.1)
- added REF**: MountingHole_3.2mm_M3_ISO7380_Pad, MountingHole:MountingHole_3.2mm_M3_ISO7380_Pad, F.Cu at (136.0, 151.3)
- added REF**: MountingHole_3.2mm_M3_ISO7380_Pad, MountingHole:MountingHole_3.2mm_M3_ISO7380_Pad, F.Cu at (136.0, 229.1)
- added REF**: MountingHole_3.2mm_M3_ISO7380_Pad, MountingHole:MountingHole_3.2mm_M3_ISO7380_Pad, F.Cu at (68.8, 177.2)
- added REF**: MountingHole_3.2mm_M3_ISO7380_Pad, MountingHole:MountingHole_3.2mm_M3_ISO7380_Pad, F.Cu at (68.7, 202.9)
- added REF**: MountingHole_3.2mm_M3_ISO7380_Pad, MountingHole:MountingHole_3.2mm_M3_ISO7380_Pad, F.Cu at (68.7, 151.3)
- C1: moved to B.Cu
- C2: value CP -> 100uF
- D1: footprint Diode_THT:D_DO-41_SOD81_P10.16mm_Horizontal -> Diode_THT:D_DO-41_SOD81_P12.70mm_Horizontal; moved to B.Cu
- D2: footprint Diode_THT:D_DO-41_SOD81_P10.16mm_Horizontal -> Diode_THT:D_DO-41_SOD81_P12.70mm_Horizontal
- J1: value Regular -> Spare1; footprint Connector_USB:USB3_A_Molex_48393-001 -> Connector_Phoenix_MC:PhoenixContact_MCV_1,5_2-G-3.5_1x02_P3.50mm_Vertical
- J2: value Regular -> Spare2; footprint Connector_USB:USB3_A_Molex_48393-001 -> Connector_Phoenix_MC:PhoenixContact_MCV_1,5_2-G-3.5_1x02_P3.50mm_Vertical
- J3: value Accelerated -> Regular; footprint Connector_USB:USB3_A_Molex_48393-001 -> Connector_Phoenix_MC:PhoenixContact_MCV_1,5_2-G-3.5_1x02_P3.50mm_Vertical
- J4: value Fast -> Regular; footprint Connector_USB:USB3_A_Molex_48393-001 -> Connector_Phoenix_MC:PhoenixContact_MCV_1,5_2-G-3.5_1x02_P3.50mm_Vertical
- J6: value USB_OTG -> USB_B PTH Receptable; footprint Connector_USB:USB_Micro-B_Wuerth_629105150521_CircularHoles -> Connector_USB:USB_B_OST_USB-B1HSxx_Horizontal
- J7: value SIL10 -> Serial 7 Segment Display
- P10, P11, P5, P9: footprint Connector_Wire:SolderWirePad_1x02_P5.08mm_Drill1.5mm -> Connector_PinSocket_2.54mm:PinSocket_1x02_P2.54mm_Vertical; moved to B.Cu
- P2: value CONN_2 -> POWER_DELIVERY; footprint Connector_Wire:SolderWirePad_1x02_P5.08mm_Drill1.5mm -> Connector_Phoenix_MC:PhoenixContact_MCV_1,5_2-G-3.5_1x02_P3.50mm_Vertical
- P3, P6, P7, P8: footprint Connector_Wire:SolderWirePad_1x02_P5.08mm_Drill1.5mm -> Connector_Phoenix_MC:PhoenixContact_MCV_1,5_2-G-3.5_1x02_P3.50mm_Vertical
- P4: footprint Connector_Wire:SolderWirePad_1x04_P3.81mm_Drill1mm -> Connector_PinSocket_2.54mm:PinSocket_1x04_P2.54mm_Vertical; moved to B.Cu
- R1, R11: footprint Resistor_THT:R_Axial_Power_L50.0mm_W9.0mm_P55.88mm -> Resistor_THT:R_Axial_Power_L48.0mm_W12.5mm_P55.88mm; moved to B.Cu
- R10, R6: value 500Ω 0.1W -> 500Ω 1% 0.1W; footprint Resistor_THT:R_Axial_DIN0204_L3.6mm_D1.6mm_P7.62mm_Horizontal -> Resistor_THT:R_Axial_DIN0207_L6.3mm_D2.5mm_P15.24mm_Horizontal; moved to B.Cu
- R12: value R -> 0; footprint Resistor_THT:R_Axial_DIN0309_L9.0mm_D3.2mm_P12.70mm_Horizontal -> Resistor_THT:R_Axial_DIN0207_L6.3mm_D2.5mm_P15.24mm_Horizontal
- R2: footprint Resistor_THT:R_Axial_Power_L50.0mm_W9.0mm_P55.88mm -> Resistor_THT:R_Axial_DIN0516_L15.5mm_D5.0mm_P25.40mm_Horizontal; moved to B.Cu
- R3, R4, R5, R9: footprint Resistor_THT:R_Axial_DIN0204_L3.6mm_D1.6mm_P7.62mm_Horizontal -> Resistor_THT:R_Axial_DIN0207_L6.3mm_D2.5mm_P10.16mm_Horizontal; moved to B.Cu
- R7: value 100Ω 0.5W -> 100Ω 1% 1W; footprint Resistor_THT:R_Axial_Power_L50.0mm_W9.0mm_P55.88mm -> Resistor_THT:R_Axial_DIN0516_L15.5mm_D5.0mm_P25.40mm_Horizontal; moved to B.Cu
- R8: value 33Ω 1.5W -> 33Ω 1% 3W; footprint Resistor_THT:R_Axial_Power_L50.0mm_W9.0mm_P55.88mm -> Resistor_THT:R_Axial_DIN0614_L14.3mm_D5.7mm_P25.40mm_Horizontal; moved to B.Cu
- moved R5 189.4 mm to (97.3, 148.1), turned to 180 degrees
- moved D5 182.2 mm to (101.1, 151.3)
- moved R3 177.5 mm to (106.8, 208.0), turned to 180 degrees
- moved D3 174.9 mm to (101.1, 202.9)
- moved R8 172.0 mm to (115.1, 157.6)
- moved P6 172.0 mm to (80.1, 201.0), turned to 270 degrees
- moved R6 170.4 mm to (109.3, 211.8)
- moved P3 162.9 mm to (80.1, 227.2), turned to 270 degrees
- moved P8 152.4 mm to (80.1, 149.4), turned to 270 degrees
- moved D6 151.6 mm to (101.1, 229.1)
- moved P7 144.1 mm to (80.3, 175.3), turned to 270 degrees
- moved R9 143.6 mm to (106.8, 234.2), turned to 180 degrees
- moved R4 137.8 mm to (103.8, 173.4), turned to 180 degrees
- moved R10 132.3 mm to (109.3, 238.0), turned to 180 degrees
- moved D4 126.2 mm to (101.2, 177.2)
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Connections:
- net /DisplayRx renamed SW_UART_DISPLAY
- net /Vh10 renamed ADC_IN0
- J1 pad 2: (no net) -> Net-(J1-Pad2)
- J2 pad 2: (no net) -> Net-(J2-Pad2)
- J3 pad 2: (no net) -> Net-(J3-Pad2)
- J4 pad 2: (no net) -> Net-(J4-Pad2)
- J6 pad 4: (no net) -> GND
- J7 pad 10: (no net) -> Net-(J7-Pad10)
- J7 pad 2: (no net) -> Net-(J7-Pad2)
- J7 pad 3: (no net) -> Net-(J7-Pad3)
- J7 pad 4: (no net) -> Net-(J7-Pad4)
- J7 pad 5: (no net) -> Net-(J7-Pad5)
- J7 pad 6: (no net) -> Net-(J7-Pad6)
- J7 pad 9: (no net) -> Net-(J7-Pad9)
- R12 pad 1: Net-(P12-Pad2) -> Net-(R12-Pad1)
- R12 pad 2: Net-(P12-Pad2) -> Net-(J1-Pad2)
- U1 pad 1: GND -> Net-(U1-Pad1)
- U1 pad 11: Net-(J1-Pad4) -> Net-(J3-Pad2)
- U1 pad 12: Net-(J2-Pad4) -> Net-(J4-Pad2)
- U1 pad 13: Net-(J3-Pad4) -> Net-(J8-Pad2)
- U1 pad 14: Net-(J4-Pad4) -> Net-(J9-Pad2)
- U1 pad 15: Net-(P12-Pad2) -> Net-(R12-Pad1)
- U1 pad 17: (no net) -> Net-(R14-Pad1)
- U1 pad 18: (no net) -> Net-(R15-Pad1)
- U1 pad 2: GND -> Net-(U1-Pad2)
- U2 pad 1: (no net) -> Net-(U2-Pad1)
- U2 pad 12: (no net) -> Net-(U1-Pad2)
- U2 pad 15: (no net) -> Net-(U2-Pad15)
- U2 pad 17: (no net) -> Net-(U2-Pad17)
- U2 pad 18: (no net) -> Net-(U2-Pad18)
- U2 pad 2: (no net) -> Net-(U2-Pad2)
- U2 pad 20: (no net) -> Net-(U2-Pad20)
- U2 pad 21: (no net) -> Net-(U2-Pad21)
- U2 pad 22: (no net) -> Net-(U2-Pad22)
- U2 pad 23: (no net) -> Net-(U2-Pad23)
- U2 pad 24: (no net) -> Net-(U2-Pad24)
- U2 pad 25: (no net) -> Net-(U2-Pad25)
- U2 pad 26: (no net) -> Net-(U1-Pad1)
- U2 pad 3: RESET_SW -> Net-(U2-Pad3)
- U2 pad 30: (no net) -> Net-(U2-Pad30)
Routing:
- net +5V: track 0.00 -> 352.9 mm, vias 0 -> 3
- net START_SW: track 0.00 -> 149.1 mm, vias 0 -> 2
- net Net-(J9-Pad2): track 0.00 -> 123.6 mm
- net RESET_SW: track 0.00 -> 93.7 mm
- net Net-(J4-Pad2): track 0.00 -> 85.0 mm
- net SW_UART_DISPLAY: track 0.00 -> 79.5 mm, vias 0 -> 2
- net ADC_IN0: track 0.00 -> 79.0 mm
- net Net-(J3-Pad2): track 0.00 -> 75.3 mm
- net Net-(J8-Pad2): track 0.00 -> 63.4 mm, vias 0 -> 2
- net Net-(U1-Pad1): track 0.00 -> 62.6 mm
- net /Vharvest: track 0.00 -> 34.4 mm
- net Net-(R12-Pad1): track 0.00 -> 29.4 mm
- net Net-(R13-Pad1): track 0.00 -> 28.8 mm
- net /Charging stations/POWER_5V_S4: track 0.00 -> 25.4 mm
- net /Charging stations/POWER_5V_S1: track 0.00 -> 25.0 mm
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- added copper zone on B.Cu, net /Charging stations/POWER_GND_S1
- added copper zone on B.Cu, net /Charging stations/POWER_GND_S2
- added copper zone on B.Cu, net /Charging stations/POWER_GND_S3
- added copper zone on B.Cu, net /Charging stations/POWER_GND_S4
- added copper zone on B.Cu, net GND
- added copper zone on F.Cu, net GND
Other:
- board size 259.1 x 109.2 mm -> 105.4 x 200.8 mm
- net class esigelec added: clearance 0.5, trace_width 0.8, via_dia 1.2, via_drill 0.8
- board text added: "+"
- board text added: "1"
- board text added: "100mm"
- board text added: "ACCEL"
- board text added: "Accelerated source"
- board text added: "DELIVERY"
- board text added: "FAST"
- board text added: "REGULAR"
- board text added: "Regular source"
- board text added: "U"
- board text added: "bottom"
- board text added: "top"
- board text removed: "Sources PVC Tube, 20cm height, 8cm diameter (7.2 inner)"

Commit message: Deleted useless component (C), minor changes after tests
Parts:
- removed C1: 10uF, Capacitor_THT:C_Rect_L26.5mm_W8.5mm_P22.50mm_MKS4
Connections:
- J7 pad 10: Net-(J7-Pad10) -> (no net)
- J7 pad 2: Net-(J7-Pad2) -> (no net)
- J7 pad 3: Net-(J7-Pad3) -> (no net)
- J7 pad 4: Net-(J7-Pad4) -> (no net)
- J7 pad 5: Net-(J7-Pad5) -> (no net)
- J7 pad 6: Net-(J7-Pad6) -> (no net)
- J7 pad 9: Net-(J7-Pad9) -> (no net)
- U2 pad 1: Net-(U2-Pad1) -> (no net)
- U2 pad 15: Net-(U2-Pad15) -> (no net)
- U2 pad 17: Net-(U2-Pad17) -> (no net)
- U2 pad 18: Net-(U2-Pad18) -> (no net)
- U2 pad 2: Net-(U2-Pad2) -> (no net)
- U2 pad 20: Net-(U2-Pad20) -> (no net)
- U2 pad 21: Net-(U2-Pad21) -> (no net)
- U2 pad 22: Net-(U2-Pad22) -> (no net)
- U2 pad 23: Net-(U2-Pad23) -> (no net)
- U2 pad 24: Net-(U2-Pad24) -> (no net)
- U2 pad 25: Net-(U2-Pad25) -> (no net)
- U2 pad 3: Net-(U2-Pad3) -> (no net)
- U2 pad 30: Net-(U2-Pad30) -> (no net)
Routing:
- net ADC_IN0: track 79.0 -> 73.4 mm

Commit message: Last changes on the PCB before production
Parts:
- moved D4 2.55 mm to (101.5, 179.7)
- moved P10 2.55 mm to (121.8, 181.6)
- moved P7 2.55 mm to (80.5, 177.8)
- moved R10 2.55 mm to (109.6, 240.5)
- moved R4 2.55 mm to (104.0, 175.9)
- moved R5 2.55 mm to (97.5, 150.6)
- moved R9 2.55 mm to (107.1, 236.7)
- moved P5 2.55 mm to (121.7, 232.9)
- moved REF** 2.55 mm to (136.4, 179.7)
- moved REF** 2.55 mm to (69.1, 179.7)
- moved D3 2.55 mm to (101.3, 205.5)
- moved D5 2.55 mm to (101.3, 153.8)
- moved D6 2.55 mm to (101.3, 231.6)
- moved P3 2.55 mm to (80.4, 229.7)
- moved P6 2.55 mm to (80.4, 203.6)
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Routing:
- net Net-(J3-Pad2): track 75.3 -> 71.6 mm
- net Net-(J8-Pad2): track 63.4 -> 59.8 mm
- net Net-(J9-Pad2): track 123.6 -> 120.5 mm
- net START_SW: track 149.1 -> 147.2 mm
- net Net-(J4-Pad2): track 85.0 -> 83.2 mm
Other:
- board size 105.4 x 200.8 mm -> 105.4 x 203.3 mm
